File: sleep_rig_controller_5x3.kicad_pcb (KiCad board)
At the start: 2 copper layers, 121.3 x 67.3 mm, 39 parts, among them J1 M12-5_RCPT_F, J2 M12-5_RCPT_F, J3 DB9F, J4 DB9M, P1 MINI_FIT_JR_02X03_M_RA, P2 PWR_JACK_2.5x5.5, U1 SN74ABT541BDWR, U2 SN74ABT541BDWR

Commit message: smart_vision -> sleep_rig.
Parts:
- C1, C2, C3, C4, C5, C6, R1, R2, R3, R4, R5, R6, R7, R8: footprint smart_vision_controller_5x3:SM1210 -> sleep_rig_controller_5x3:SM1210
- D1: footprint smart_vision_controller_5x3:CFP15 -> sleep_rig_controller_5x3:CFP15
- HPS1, HPS2, HPS3, HPS4: footprint smart_vision_controller_5x3:PG-TO252-5-11 -> sleep_rig_controller_5x3:PG-TO252-5-11
- J1, J2: footprint smart_vision_controller_5x3:M12-5_RCPT_F -> sleep_rig_controller_5x3:M12-5_RCPT_F
- J3: footprint smart_vision_controller_5x3:DB9F -> sleep_rig_controller_5x3:DB9F
- J4: footprint smart_vision_controller_5x3:DB9M -> sleep_rig_controller_5x3:DB9M
- L1: footprint smart_vision_controller_5x3:LED_555-3XXX_R -> sleep_rig_controller_5x3:LED_555-3XXX_R
- L10, L11, L2, L3, L4, L5, L6, L7, L8, L9: footprint smart_vision_controller_5x3:LED_555-3XXX_G -> sleep_rig_controller_5x3:LED_555-3XXX_G
- MDB1: footprint smart_vision_controller_5x3:MODULAR_DEVICE_BASE_5X3_MALE -> sleep_rig_controller_5x3:MODULAR_DEVICE_BASE_5X3_MALE
- P1: footprint smart_vision_controller_5x3:MINI-FIT-JR_02X03_M_RA -> sleep_rig_controller_5x3:MINI-FIT-JR_02X03_M_RA
- P2: footprint smart_vision_controller_5x3:DCJACK_2PIN_HIGHCURRENT -> sleep_rig_controller_5x3:DCJACK_2PIN_HIGHCURRENT
- U1, U2: footprint smart_vision_controller_5x3:SOIC_20 -> sleep_rig_controller_5x3:SOIC_20
Other:
- board text added: "Janelia Modular Device sleep_rig_controller part_number: 1270 08/2018 ver 1.0 5x3"
- board text removed: "Janelia Modular Device smart_vision_controller part_number: 1270 08/2018 ver 1.0 5x3"
Changed lines of the file:
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@@
   (page A4)
   (title_block
-    (title smart_vision_controller_5x3)
+    (title sleep_rig_controller_5x3)
     (rev 1.0)
   )
@@
     (add_net VAA)
   )
-  (module smart_vision_controller_5x3:SM1210 (layer B.Cu)
+  (module sleep_rig_controller_5x3:SM1210 (layer B.Cu)
     (at 133.35 111.125)
     (tags "CMS SM")
@@
     )
   )
-  (module smart_vision_controller_5x3:DCJACK_2PIN_HIGHCURRENT (layer F.Cu)
+  (module sleep_rig_controller_5x3:DCJACK_2PIN_HIGHCURRENT (layer F.Cu)
     (at 190.5 118.11 270)
     (fp_text reference P2 (at -6.985 2.54) (layer F.SilkS)
@@
     (pad "" thru_hole circle (at 0 2.9972 270) (size 1.9304 1.9304) (drill 1.6002) (layers *.Cu *.Mask))
   )
-  (module smart_vision_controller_5x3:MINI-FIT-JR_02X03_M_RA (layer F.Cu)
+  (module sleep_rig_controller_5x3:MINI-FIT-JR_02X03_M_RA (layer F.Cu)
     (at 187.96 92.71 90)
     (fp_text reference P1 (at -8.255 0 180) (layer F.SilkS)
@@
     (pad "" thru_hole circle (at 4.2 0 90) (size 4 4) (drill 3) (layers *.Cu *.Mask))
   )
-  (module smart_vision_controller_5x3:MODULAR_DEVICE_BASE_5X3_MALE (layer F.Cu)
+  (module sleep_rig_controller_5x3:MODULAR_DEVICE_BASE_5X3_MALE (layer F.Cu)
     (at 91.44 105.41)
     (fp_text reference MDB1 (at 0 0) (layer F.SilkS) hide
@@
       (net 2 GND))
   )
-  (module smart_vision_controller_5x3:CFP15 (layer B.Cu)
+  (module sleep_rig_controller_5x3:CFP15 (layer B.Cu)
     (at 81.915 79.375 90)
     (fp_text reference D1 (at 0 -4.6 90) (layer B.SilkS)
@@
       (net 3 VDD) (solder_mask_margin 0.1) (clearance 0.1))
   )
-  (module smart_vision_controller_5x3:SM1210 (layer B.Cu)
+  (module sleep_rig_controller_5x3:SM1210 (layer B.Cu)
     (at 111.76 113.665)
     (tags "CMS SM")
@@
     )
   )
-  (module smart_vision_controller_5x3:SM1210 (layer B.Cu)
+  (module sleep_rig_controller_5x3:SM1210 (layer B.Cu)
     (at 143.51 113.665)
     (tags "CMS SM")
@@
     )
   )
-  (module smart_vision_controller_5x3:SM1210 (layer B.Cu)
+  (module sleep_rig_controller_5x3:SM1210 (layer B.Cu)
     (at 77.47 86.36 90)
     (tags "CMS SM")
@@
     )
   )
-  (module smart_vision_controller_5x3:SM1210 (layer B.Cu)
+  (module sleep_rig_controller_5x3:SM1210 (layer B.Cu)
     (at 77.47 99.06 90)
     (tags "CMS SM")
@@
     )
   )
-  (module smart_vision_controller_5x3:SM1210 (layer B.Cu)
+  (module sleep_rig_controller_5x3:SM1210 (layer B.Cu)
     (at 77.47 111.76 90)
     (tags "CMS SM")
@@
     )
   )
-  (module smart_vision_controller_5x3:SM1210 (layer B.Cu)
+  (module sleep_rig_controller_5x3:SM1210 (layer B.Cu)
     (at 77.47 124.46 90)
     (tags "CMS SM")
@@
     )
   )
-  (module smart_vision_controller_5x3:PG-TO252-5-11 (layer B.Cu)
+  (module sleep_rig_controller_5x3:PG-TO252-5-11 (layer B.Cu)
     (at 80.645 86.36 90)
     (fp_text reference HPS1 (at -4.445 5.1) (layer B.SilkS)
@@
       (net 2 GND))
   )
-  (module smart_vision_controller_5x3:PG-TO252-5-11 (layer B.Cu)
+  (module sleep_rig_controller_5x3:PG-TO252-5-11 (layer B.Cu)
     (at 80.645 99.06 90)
     (fp_text reference HPS2 (at -4.445 5.1) (layer B.SilkS)
@@
       (net 2 GND))
   )
-  (module smart_vision_controller_5x3:PG-TO252-5-11 (layer B.Cu)
+  (module sleep_rig_controller_5x3:PG-TO252-5-11 (layer B.Cu)
     (at 80.645 111.76 90)
     (fp_text reference HPS3 (at -4.445 5.1) (layer B.SilkS)
@@
       (net 2 GND))
   )
-  (module smart_vision_controller_5x3:PG-TO252-5-11 (layer B.Cu)
+  (module sleep_rig_controller_5x3:PG-TO252-5-11 (layer B.Cu)
     (at 80.645 124.46 90)
     (fp_text reference HPS4 (at -4.445 5.08) (layer B.SilkS)
@@
       (net 2 GND))
   )
-  (module smart_vision_controller_5x3:DB9F (layer F.Cu)
+  (module sleep_rig_controller_5x3:DB9F (layer F.Cu)
     (at 120.65 92.71)
     (fp_text reference J3 (at 0 7.62) (layer F.SilkS)
@@
       (net 18 /BUZZER))
   )
-  (module smart_vision_controller_5x3:DB9M (layer F.Cu)
+  (module sleep_rig_controller_5x3:DB9M (layer F.Cu)
     (at 120.65 118.11)
     (fp_text reference J4 (at 0 -7.62) (layer F.SilkS)
@@
       (net 2 GND))
   )
-  (module smart_vision_controller_5x3:M12-5_RCPT_F (layer F.Cu)
+  (module sleep_rig_controller_5x3:M12-5_RCPT_F (layer F.Cu)
     (at 152.4 92.71)
     (fp_text reference J1 (at 0 10.16) (layer F.SilkS)
@@
       (net 4 VAA))
   )
-  (module smart_vision_controller_5x3:M12-5_RCPT_F (layer F.Cu)
+  (module sleep_rig_controller_5x3:M12-5_RCPT_F (layer F.Cu)
     (at 152.4 118.11)
     (fp_text reference J2 (at 0 -10.16) (layer F.SilkS)
@@
       (net 4 VAA))
   )
-  (module smart_vision_controller_5x3:SM1210 (layer B.Cu)
+  (module sleep_rig_controller_5x3:SM1210 (layer B.Cu)
     (at 73.025 85.725 180)
     (tags "CMS SM")
@@
     )
   )
-  (module smart_vision_controller_5x3:SM1210 (layer B.Cu)
+  (module sleep_rig_controller_5x3:SM1210 (layer B.Cu)
     (at 73.025 99.06 180)
     (tags "CMS SM")
@@
     )
   )
-  (module smart_vision_controller_5x3:SM1210 (layer B.Cu)
+  (module sleep_rig_controller_5x3:SM1210 (layer B.Cu)
     (at 73.025 111.76 180)
     (tags "CMS SM")
@@
     )
   )
-  (module smart_vision_controller_5x3:SM1210 (layer B.Cu)
+  (module sleep_rig_controller_5x3:SM1210 (layer B.Cu)
     (at 73.025 124.46 180)
     (tags "CMS SM")
@@
     )
   )
-  (module smart_vision_controller_5x3:SM1210 (layer B.Cu)
+  (module sleep_rig_controller_5x3:SM1210 (layer B.Cu)
     (at 133.35 99.695)
     (tags "CMS SM")
@@
     )
   )
-  (module smart_vision_controller_5x3:SM1210 (layer B.Cu)
+  (module sleep_rig_controller_5x3:SM1210 (layer B.Cu)
     (at 133.35 103.505)
     (tags "CMS SM")
@@
     )
   )
-  (module smart_vision_controller_5x3:SM1210 (layer B.Cu)
+  (module sleep_rig_controller_5x3:SM1210 (layer B.Cu)
     (at 133.35 107.315)
     (tags "CMS SM")
@@
     )
   )
-  (module smart_vision_controller_5x3:SOIC_20 (layer B.Cu)
+  (module sleep_rig_controller_5x3:SOIC_20 (layer B.Cu)
     (at 111.76 105.41 180)
     (fp_text reference U1 (at 0 7.62 180) (layer B.SilkS)
@@
       (net 1 VEE) (solder_mask_margin 0.07) (clearance 0.07))
   )
-  (module smart_vision_controller_5x3:SOIC_20 (layer B.Cu)
+  (module sleep_rig_controller_5x3:SOIC_20 (layer B.Cu)
     (at 143.51 105.41 180)
     (fp_text reference U2 (at 0 7.62 180) (layer B.SilkS)
@@
       (net 1 VEE) (solder_mask_margin 0.07) (clearance 0.07))
   )
-  (module smart_vision_controller_5x3:LED_555-3XXX_R (layer F.Cu)
+  (module sleep_rig_controller_5x3:LED_555-3XXX_R (layer F.Cu)
     (at 166.37 105.41)
     (fp_text reference L1 (at 0 -4.445 180) (layer F.SilkS)
@@
       (net 2 GND))
   )
-  (module smart_vision_controller_5x3:LED_555-3XXX_G (layer F.Cu)
+  (module sleep_rig_controller_5x3:LED_555-3XXX_G (layer F.Cu)
     (at 93.345 86.995)
     (fp_text reference L2 (at -1.905 0 90) (layer F.SilkS)
@@
       (net 28 /C_0))
   )
-  (module smart_vision_controller_5x3:LED_555-3XXX_G (layer F.Cu)
+  (module sleep_rig_controller_5x3:LED_555-3XXX_G (layer F.Cu)
     (at 95.885 86.995)
     (fp_text reference L3 (at 0 4.5) (layer F.SilkS) hide
@@
       (net 2 GND))
   )
-  (module smart_vision_controller_5x3:LED_555-3XXX_G (layer F.Cu)
+  (module sleep_rig_controller_5x3:LED_555-3XXX_G (layer F.Cu)
     (at 98.425 86.995)
     (fp_text reference L4 (at 0 4.5) (layer F.SilkS) hide
@@
       (net 30 /C_2))
   )
-  (module smart_vision_controller_5x3:LED_555-3XXX_G (layer F.Cu)
+  (module sleep_rig_controller_5x3:LED_555-3XXX_G (layer F.Cu)
     (at 100.965 86.995)
     (fp_text reference L5 (at 1.905 0 90) (layer F.SilkS)
@@
       (net 2 GND))
   )
-  (module smart_vision_controller_5x3:LED_555-3XXX_G (layer F.Cu)
+  (module sleep_rig_controller_5x3:LED_555-3XXX_G (layer F.Cu)
     (at 93.345 123.825)
     (fp_text reference L6 (at -1.905 0 90) (layer F.SilkS)
@@
       (net 32 /C_8))
   )
-  (module smart_vision_controller_5x3:LED_555-3XXX_G (layer F.Cu)
+  (module sleep_rig_controller_5x3:LED_555-3XXX_G (layer F.Cu)
     (at 95.885 123.825)
     (fp_text reference L7 (at 0 4.5) (layer F.SilkS) hide
@@
       (net 33 /C_9))
   )
-  (module smart_vision_controller_5x3:LED_555-3XXX_G (layer F.Cu)
+  (module sleep_rig_controller_5x3:LED_555-3XXX_G (layer F.Cu)
     (at 98.425 123.825)
     (fp_text reference L8 (at 0 4.5) (layer F.SilkS) hide
@@
       (net 2 GND))
   )
-  (module smart_vision_controller_5x3:LED_555-3XXX_G (layer F.Cu)
+  (module sleep_rig_controller_5x3:LED_555-3XXX_G (layer F.Cu)
     (at 100.965 123.825)
     (fp_text reference L9 (at 1.905 0 90) (layer F.SilkS)
@@
       (net 2 GND))
   )
-  (module smart_vision_controller_5x3:LED_555-3XXX_G (layer F.Cu)
+  (module sleep_rig_controller_5x3:LED_555-3XXX_G (layer F.Cu)
     (at 141.605 86.995)
     (fp_text reference L10 (at 1.905 0 90) (layer F.SilkS)
@@
       (net 2 GND))
   )
-  (module smart_vision_controller_5x3:LED_555-3XXX_G (layer F.Cu)
+  (module sleep_rig_controller_5x3:LED_555-3XXX_G (layer F.Cu)
     (at 141.605 123.825)
     (fp_text reference L11 (at 1.905 -0.635 90) (layer F.SilkS)
@@
     (effects (font (size 1.016 1.016) (thickness 0.1905)))
   )
-  (gr_text "Janelia Modular Device\nsmart_vision_controller\npart_number: 1270\n08/2018 ver 1.0 5x3" (at 73.66 105.41 90) (layer F.SilkS)
+  (gr_text "Janelia Modular Device\nsleep_rig_controller\npart_number: 1270\n08/2018 ver 1.0 5x3" (at 73.66 105.41 90) (layer F.SilkS)
     (effects (font (size 1.016 1.016) (thickness 0.254)))
   )
