File: backlight_controller_5x3.kicad_pcb (KiCad board)
At the start: 2 copper layers, 121.3 x 67.3 mm, 50 parts, among them J1 DB9F_SMD, J10 M12-5_RCPT_F, J2 DB9M_SMD, J3 M12-5_RCPT_F, J4 M12-5_RCPT_F, J5 M12-5_RCPT_F, J6 M12-5_RCPT_F, J7 M12-5_RCPT_F, J8 M12-5_RCPT_F, J9 M12-5_RCPT_F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

Commit message: Changes towards v1.1.
Routing:
- net GND: track 557.6 -> 0.00 mm, vias 1 -> 0
- net VAA: track 312.1 -> 0.00 mm, vias 2 -> 0
- net VEE: track 150.4 -> 0.00 mm, vias 1 -> 0
- net VDD: track 121.9 -> 0.00 mm, vias 2 -> 0
- net /CHANNEL_15: track 106.4 -> 0.00 mm, vias 1 -> 0
- net /CHANNEL_11: track 100.1 -> 0.00 mm, vias 1 -> 0
- net /CHANNEL_8: track 93.7 -> 0.00 mm, vias 1 -> 0
- net /~ENABLE: track 88.8 -> 0.00 mm, vias 3 -> 0
- net /backlight_5x3/C_0: track 80.3 -> 0.00 mm
- net /CHANNEL_13: track 79.0 -> 0.00 mm, vias 2 -> 0
- net /CHANNEL_12: track 78.3 -> 0.00 mm, vias 2 -> 0
- net /CHANNEL_14: track 77.4 -> 0.00 mm, vias 2 -> 0
- net /backlight_5x3/high_power_outputs/OUTPUT_2: track 73.2 -> 0.00 mm, vias 1 -> 0
- net /backlight_5x3/C_3: track 72.2 -> 0.00 mm
- net /backlight_5x3/C_1: track 68.3 -> 0.00 mm
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- removed copper zone on B.Cu, net GND
- removed copper zone on F.Cu, net VAA
Other:
- board text added: "Janelia Modular Device backlight_controller part_number: 1270 10/2018 ver 1.1 5x3"
- board text removed: "Janelia Modular Device backlight_controller part_number: 1270 09/2018 ver 1.0 5x3"
