File: backlight_controller_5x3.kicad_pcb (KiCad board)
At the start: 2 copper layers, 121.3 x 67.3 mm, 84 parts, among them J1 HEADER_01x25_MALE, J10 M12-5-RCPT, J11 M12-5-RCPT, J12 M12-5-RCPT, J2 HEADER_01x25_MALE, J3 DB9F, J4 DB9M, J5 M12-5-RCPT, J6 M12-5-RCPT, J7 M12-5-RCPT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

Commit message: Fix missing component field values
Parts:
- J1, J2: value HEADER_01x25_MALE -> HEADER_01X25_MALE
Connections:
- HPS1 pad 4: (no net) -> Net-(HPS1-Pad4)
- HPS2 pad 4: (no net) -> Net-(HPS2-Pad4)
- HPS3 pad 4: (no net) -> Net-(HPS3-Pad4)
- HPS4 pad 4: (no net) -> Net-(HPS4-Pad4)
- J1 pad 11: (no net) -> /D40
- J1 pad 12: (no net) -> /D41
- J1 pad 13: (no net) -> /D42
- J1 pad 14: (no net) -> /D11.MOSI0
- J1 pad 15: (no net) -> /D12.MISO0
- J1 pad 16: (no net) -> /D50.A24
- J1 pad 17: (no net) -> /D49.A23
- J1 pad 18: (no net) -> /D48.TX6.SDA0B
- J1 pad 19: (no net) -> /D47.RX6.SCLOB
- J1 pad 20: (no net) -> /D43.CS2
- J1 pad 21: (no net) -> /D44.MOSI2
- J1 pad 24: (no net) -> /D45.MISO2
- J1 pad 25: (no net) -> /D46.SCK2
- J1 pad 3: (no net) -> /A10
- J1 pad 4: (no net) -> /A11
- J1 pad 6: (no net) -> /D55
- J1 pad 7: (no net) -> /D54.CS2
- J10 pad 4: (no net) -> Net-(J10-Pad4)
- J11 pad 4: (no net) -> Net-(J11-Pad4)
- J12 pad 4: (no net) -> Net-(J12-Pad4)
- J2 pad 1: (no net) -> /AREF
- J2 pad 11: (no net) -> /D17.A3.SDA0B
- J2 pad 12: (no net) -> /D16.A2.SCL0B
- J2 pad 13: (no net) -> /D15.A1.CS0
- J2 pad 15: (no net) -> /D13.LED.SCK0
- J2 pad 16: (no net) -> /D53.SCK2B
- J2 pad 17: (no net) -> /A22.DAC1
- J2 pad 18: (no net) -> /A21.DAC0
- J2 pad 19: (no net) -> /D51.MISO2B
- J2 pad 24: (no net) -> /D34.A15.SDA0B.RX5
- J2 pad 25: (no net) -> /D33.A14.SCL0B.TX5
- J2 pad 3: (no net) -> /AGND
- J2 pad 4: (no net) -> /3.3V_250mA
- J5 pad 4: (no net) -> Net-(J5-Pad4)
- J6 pad 4: (no net) -> Net-(J6-Pad4)
- J7 pad 4: (no net) -> Net-(J7-Pad4)
- J8 pad 4: (no net) -> Net-(J8-Pad4)
- J9 pad 4: (no net) -> Net-(J9-Pad4)
- MH1 pad 1: (no net) -> Net-(MH1-Pad1)
- MH2 pad 1: (no net) -> Net-(MH2-Pad1)
- MH3 pad 1: (no net) -> Net-(MH3-Pad1)
- MH4 pad 1: (no net) -> Net-(MH4-Pad1)
